Commit message: Completed Robotmodel

File: src/kuka_description/urdf/robot.urdf (robot description, URDF)
Before this commit: robot robot, 9 links, 8 joints
Links:
- link base_link: geometry collision mesh filename=package://kuka_description/meshes/kuka_kr5_arc/visual/Baseb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 scale=.001 .001 .001; visual mesh filename=package://kuka_description/meshes/kuka_kr5_arc/visual/Baseb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 scale=.001 .001 .001
- link link1: geometry collision mesh filename=package://kuka_description/meshes/kuka_kr5_arc/visual/Link1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 scale=.004 .004 .004; visual mesh filename=package://kuka_description/meshes/kuka_kr5_arc/visual/Link1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 scale=.004 .004 .004
